File: dipext-pin_r4/dipext-pin_r4.kicad_pcb (KiCad board)
At the start: 2 copper layers, 88.9 x 88.9 mm, 16 parts, among them J1 ZIF, J2 IDC40, J3 Conn_02x20_Odd_Even, J4 Conn_02x20_Odd_Even

Commit message: Yes.
Parts:
- added J5: 01x20, Connector_PinHeader_2.54mm:PinHeader_1x20_P2.54mm_Vertical, F.Cu at (87.4, 46.5)
- added J6: 01x20, Connector_PinHeader_2.54mm:PinHeader_1x20_P2.54mm_Vertical, F.Cu at (77.5, 46.5)
- added J7: 01x20, Connector_PinHeader_2.54mm:PinHeader_1x20_P2.54mm_Vertical, F.Cu at (41.7, 46.4)
- added J8: 01x20, Connector_PinHeader_2.54mm:PinHeader_1x20_P2.54mm_Vertical, F.Cu at (51.5, 46.4)
- moved J4 2.47 mm to (81.2, 46.5)
- moved J1 2.35 mm to (56.9, 46.4)
- moved J3 2.25 mm to (45.4, 46.4)
- moved J2 1.71 mm to (93.1, 46.5)
Routing:
- net /P11: track 49.2 -> 52.5 mm
- net /P5: track 49.2 -> 52.5 mm
- net /P4: track 49.2 -> 52.4 mm
- net /P3: track 49.2 -> 52.4 mm
- net /P2: track 49.2 -> 52.4 mm
- net /P19: track 49.2 -> 52.4 mm
- net /P17: track 49.2 -> 52.4 mm
- net /P10: track 49.2 -> 52.4 mm
- net /P15: track 49.2 -> 52.4 mm
- net /P13: track 49.2 -> 52.4 mm
- net /P8: track 49.2 -> 52.4 mm
- net /P12: track 49.2 -> 52.4 mm
- net /P20: track 49.2 -> 52.4 mm
- net /P9: track 49.2 -> 52.4 mm
- net /P18: track 49.2 -> 52.4 mm
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Other:
- net class Default removed
- board text added: "DIP40EXT-PIN R5"
- board text added: "© 2018 JOHN MCMASTER, 2021 ANDREY T. https://spirit.re/"
- board text removed: "(C) 2018 JOHN MCMASTER"
- board text removed: "DIP40EXT-PIN R4"
