File: dipext-pin_r4/dipext-pin_r4.kicad_pcb (KiCad board)
At the start: 2 copper layers, 88.9 x 88.9 mm, 20 parts, among them J1 ZIF, J2 IDC40, J3 Conn_02x20_Odd_Even, J4 Conn_02x20_Odd_Even, J5 01x20, J6 01x20, J7 01x20, J8 01x20

Commit message: Revert "Yes."
This reverts commit 611ce2b3961d5ca419525b40e4a89030cbd90d7e.

	deleted:    dipext-pin_r4/Gerbers.zip
	deleted:    dipext-pin_r4/Gerbers/dipext-pin_r4-B_Cu.gbr
	deleted:    dipext-pin_r4/Gerbers/dipext-pin_r4-B_Mask.gbr
	deleted:    dipext-pin_r4/Gerbers/dipext-pin_r4-B_Silkscreen.gbr
	deleted:    dipext-pin_r4/Gerbers/dipext-pin_r4-Edge_Cuts.gbr
	deleted:    dipext-pin_r4/Gerbers/dipext-pin_r4-F_Cu.gbr
	deleted:    dipext-pin_r4/Gerbers/dipext-pin_r4-F_Mask.gbr
	deleted:    dipext-pin_r4/Gerbers/dipext-pin_r4-F_Silkscreen.gbr
	deleted:    dipext-pin_r4/Gerbers/dipext-pin_r4-NPTH-drl_map.ps
	deleted:    dipext-pin_r4/Gerbers/dipext-pin_r4-NPTH.drl
	deleted:    dipext-pin_r4/Gerbers/dipext-pin_r4-PTH-drl_map.ps
	deleted:    dipext-pin_r4/Gerbers/dipext-pin_r4-PTH.drl
	deleted:    dipext-pin_r4/Gerbers/dipext-pin_r4-job.gbrjob
	deleted:    dipext-pin_r4/dipext-pin_r4-rescue.lib
	modified:   dipext-pin_r4/dipext-pin_r4.kicad_pcb
	deleted:    dipext-pin_r4/dipext-pin_r4.kicad_prl
	deleted:    dipext-pin_r4/dipext-pin_r4.kicad_pro
	deleted:    dipext-pin_r4/dipext-pin_r4.kicad_sch
	new file:   dipext-pin_r4/dipext-pin_r4.zip
	deleted:    dipext-pin_r4/rescue-backup/dipext-pin_r4-2021-02-06-23-54-14.kicad_pro
	deleted:    dipext-pin_r4/rescue-backup/dipext-pin_r4-2021-02-06-23-54-14.sch
	deleted:    dipext-pin_r4/rescue-backup/dipext-pin_r4-cache-2021-02-06-23-54-14.lib
	deleted:    dipext-pin_r4/sym-lib-table
Parts:
- removed J5, J6, J7, J8: 01x20, Connector_PinHeader_2.54mm:PinHeader_1x20_P2.54mm_Vertical
- moved J4 2.47 mm to (78.7, 47.0)
- moved J1 2.35 mm to (54.6, 47.0)
- moved J3 2.25 mm to (43.2, 47.0)
- moved J2 1.71 mm to (91.4, 47.0)
Routing:
- net /P11: track 52.5 -> 49.2 mm
- net /P5: track 52.5 -> 49.2 mm
- net /P4: track 52.4 -> 49.2 mm
- net /P3: track 52.4 -> 49.2 mm
- net /P2: track 52.4 -> 49.2 mm
- net /P19: track 52.4 -> 49.2 mm
- net /P17: track 52.4 -> 49.2 mm
- net /P10: track 52.4 -> 49.2 mm
- net /P15: track 52.4 -> 49.2 mm
- net /P13: track 52.4 -> 49.2 mm
- net /P8: track 52.4 -> 49.2 mm
- net /P12: track 52.4 -> 49.2 mm
- net /P20: track 52.4 -> 49.2 mm
- net /P9: track 52.4 -> 49.2 mm
- net /P18: track 52.4 -> 49.2 mm
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Other:
- net class Default added: clearance 0.1524, trace_width 0.3048, via_dia 0.6858, via_drill 0.3302
- board text added: "(C) 2018 JOHN MCMASTER"
- board text added: "DIP40EXT-PIN R4"
- board text removed: "DIP40EXT-PIN R5"
- board text removed: "© 2018 JOHN MCMASTER, 2021 ANDREY T. https://spirit.re/"

Commit message: modified:   dipext-pin_r4/dipext-pin_r4.kicad_pcb 	modified:   dipext-pin_r4/dipext-pin_r4.kicad_prl 	modified:   dipext-pin_r4/dipext-pin_r4.kicad_pro 	modified:   dipext-pin_r5/dipext-pin_r4.kicad_prl 	modified:   dipext-pin_r5/dipext-pin_r4.kicad_pro 	modified:   dipext-pin_r5/dipext-pin_r4.kicad_sch 	modified:   simpleprobecard/Gerbers.zip 	modified:   simpleprobecard/Gerbers/simpleprobecard-B_Cu.gbr 	modified:   simpleprobecard/Gerbers/simpleprobecard-B_Mask.gbr 	modified:   simpleprobecard/Gerbers/simpleprobecard-B_Paste.gbr 	modified:   simpleprobecard/Gerbers/simpleprobecard-B_Silkscreen.gbr 	modified:   simpleprobecard/Gerbers/simpleprobecard-Edge_Cuts.gbr 	modified:   simpleprobecard/Gerbers/simpleprobecard-F_Cu.gbr 	modified:   simpleprobecard/Gerbers/simpleprobecard-F_Mask.gbr 	modified:   simpleprobecard/Gerbers/simpleprobecard-F_Paste.gbr 	modified:   simpleprobecard/Gerbers/simpleprobecard-F_Silkscreen.gbr 	modified:   simpleprobecard/Gerbers/simpleprobecard-NPTH-drl_map.ps 	modified:   simpleprobecard/Gerbers/simpleprobecard-NPTH.drl 	modified:   simpleprobecard/Gerbers/simpleprobecard-PTH-drl_map.ps 	modified:   simpleprobecard/Gerbers/simpleprobecard-PTH.drl 	modified:   simpleprobecard/Gerbers/simpleprobecard-job.gbrjob 	modified:   simpleprobecard/fp-info-cache 	modified:   simpleprobecard/simpleprobecard.kicad_pcb 	modified:   simpleprobecard/simpleprobecard.kicad_pro 	modified:   simpleprobecard/simpleprobecard.kicad_sch
Other:
- net class Default removed
