File: dipext-pin_r5/dipext-pin_r4.kicad_pcb (KiCad board)
At the start: 2 copper layers, 88.9 x 88.9 mm, 20 parts, among them J1 ZIF, J2 IDC40, J3 Conn_02x20_Odd_Even, J4 Conn_02x20_Odd_Even, J5 01x20, J6 01x20, J7 01x20, J8 01x20

Commit message: 2.54 pitch spacing
Parts:
- moved J7 1.14 mm to (42.8, 46.4)
- moved J5 1.12 mm to (86.2, 46.5)
- moved J6 1.12 mm to (78.6, 46.5)
- moved J8 1.07 mm to (50.4, 46.4)
Routing:
- net /P9: track 52.4 -> 51.2 mm
- net /P8: track 52.4 -> 51.2 mm
- net /P7: track 52.4 -> 51.2 mm
- net /P6: track 52.4 -> 51.2 mm
- net /P5: track 52.5 -> 51.3 mm
- net /P4: track 52.4 -> 51.3 mm
- net /P3: track 52.4 -> 51.3 mm
- net /P20: track 52.4 -> 51.2 mm
- net /P2: track 52.4 -> 51.3 mm
- net /P19: track 52.4 -> 51.2 mm
- net /P18: track 52.4 -> 51.2 mm
- net /P17: track 52.4 -> 51.2 mm
- net /P16: track 52.4 -> 51.2 mm
- net /P15: track 52.4 -> 51.2 mm
- net /P14: track 52.4 -> 51.2 mm
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