File: simpleprobecard/simpleprobecard.kicad_pcb (KiCad board)
At the start: 2 copper layers, 112 x 137.4 mm, 68 parts, among them J1 NEEDLES, J2 PINS

Commit message: modified:   dipext-pin_r4/dipext-pin_r4.kicad_pcb 	modified:   dipext-pin_r4/dipext-pin_r4.kicad_prl 	modified:   dipext-pin_r4/dipext-pin_r4.kicad_pro 	modified:   dipext-pin_r5/dipext-pin_r4.kicad_prl 	modified:   dipext-pin_r5/dipext-pin_r4.kicad_pro 	modified:   dipext-pin_r5/dipext-pin_r4.kicad_sch 	modified:   simpleprobecard/Gerbers.zip 	modified:   simpleprobecard/Gerbers/simpleprobecard-B_Cu.gbr 	modified:   simpleprobecard/Gerbers/simpleprobecard-B_Mask.gbr 	modified:   simpleprobecard/Gerbers/simpleprobecard-B_Paste.gbr 	modified:   simpleprobecard/Gerbers/simpleprobecard-B_Silkscreen.gbr 	modified:   simpleprobecard/Gerbers/simpleprobecard-Edge_Cuts.gbr 	modified:   simpleprobecard/Gerbers/simpleprobecard-F_Cu.gbr 	modified:   simpleprobecard/Gerbers/simpleprobecard-F_Mask.gbr 	modified:   simpleprobecard/Gerbers/simpleprobecard-F_Paste.gbr 	modified:   simpleprobecard/Gerbers/simpleprobecard-F_Silkscreen.gbr 	modified:   simpleprobecard/Gerbers/simpleprobecard-NPTH-drl_map.ps 	modified:   simpleprobecard/Gerbers/simpleprobecard-NPTH.drl 	modified:   simpleprobecard/Gerbers/simpleprobecard-PTH-drl_map.ps 	modified:   simpleprobecard/Gerbers/simpleprobecard-PTH.drl 	modified:   simpleprobecard/Gerbers/simpleprobecard-job.gbrjob 	modified:   simpleprobecard/fp-info-cache 	modified:   simpleprobecard/simpleprobecard.kicad_pcb 	modified:   simpleprobecard/simpleprobecard.kicad_pro 	modified:   simpleprobecard/simpleprobecard.kicad_sch
Parts:
- added ?: , buzzardLabel, F.Cu at (24.3, 60.0)
- added ?: , buzzardLabel, F.Cu at (19.2, 60.3)
- added ?: , buzzardLabel, F.Cu at (21.8, 60.3)
- added ?: , buzzardLabel, F.Cu at (-24.0, 60.3)
- added ?: , buzzardLabel, F.Cu at (-21.4, 69.5)
- added ?: , buzzardLabel, F.Cu at (-24.0, 69.5)
- added ?: , buzzardLabel, F.Cu at (24.3, 68.2)
- added ?: , buzzardLabel, F.Cu at (1.44, 60.3)
- added J3: Conn_02x20_Odd_Even, Connector_IDC:IDC-Header_2x20_P2.54mm_Latch_Vertical, F.Cu at (24.3, 63.7)
Connections:
- net Net-(J1-Pad1) renamed /P1
- net Net-(J1-Pad10) renamed /P10
- net Net-(J1-Pad11) renamed /P11
- net Net-(J1-Pad12) renamed /P12
- net Net-(J1-Pad13) renamed /P13
- net Net-(J1-Pad14) renamed /P14
- net Net-(J1-Pad15) renamed /P15
- net Net-(J1-Pad16) renamed /P16
- net Net-(J1-Pad17) renamed /P17
- net Net-(J1-Pad18) renamed /P18
- net Net-(J1-Pad19) renamed /P19
- net Net-(J1-Pad2) renamed /P2
- net Net-(J1-Pad20) renamed /P20
- net Net-(J1-Pad21) renamed /P21
- net Net-(J1-Pad22) renamed /P22
- net Net-(J1-Pad23) renamed /P23
- net Net-(J1-Pad24) renamed /P24
- net Net-(J1-Pad25) renamed /P25
- net Net-(J1-Pad26) renamed /P26
- net Net-(J1-Pad27) renamed /P27
- net Net-(J1-Pad28) renamed /P28
- net Net-(J1-Pad29) renamed /P29
- net Net-(J1-Pad3) renamed /P3
- net Net-(J1-Pad30) renamed /P30
- net Net-(J1-Pad31) renamed /P31
- net Net-(J1-Pad32) renamed /P32
- net Net-(J1-Pad33) renamed /P33
- net Net-(J1-Pad34) renamed /P34
- net Net-(J1-Pad35) renamed /P35
- net Net-(J1-Pad36) renamed /P36
- net Net-(J1-Pad37) renamed /P37
- net Net-(J1-Pad38) renamed /P38
- net Net-(J1-Pad39) renamed /P39
- net Net-(J1-Pad4) renamed /P4
- net Net-(J1-Pad40) renamed /P40
- net Net-(J1-Pad5) renamed /P5
- net Net-(J1-Pad6) renamed /P6
- net Net-(J1-Pad7) renamed /P7
- net Net-(J1-Pad8) renamed /P8
- net Net-(J1-Pad9) renamed /P9
Routing:
- net /P39: track 27.8 -> 126.5 mm
- net /P38: track 35.7 -> 128.2 mm
- net /P37: track 41.6 -> 134.1 mm
- net /P40: track 32.6 -> 121.6 mm
- net /P35: track 50.5 -> 136.7 mm
- net /P36: track 42.6 -> 128.8 mm
- net /P34: track 52.8 -> 132.5 mm
- net /P33: track 61.8 -> 141.2 mm
- net /P30: track 82.4 -> 155.8 mm
- net /P32: track 65.8 -> 139.0 mm
- net /P31: track 76.6 -> 149.4 mm
- net /P29: track 95.3 -> 167.8 mm
- net /P28: track 102.7 -> 169.8 mm
- net /P27: track 114.4 -> 180.5 mm
- net /P25: track 133.5 -> 195.7 mm
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