File: simpleprobecard/simpleprobecard.kicad_sch (KiCad schematic)
At the start: 8 parts, among them J1 NEEDLES, J2 PINS

Commit message: modified:   dipext-pin_r4/dipext-pin_r4.kicad_pcb 	modified:   dipext-pin_r4/dipext-pin_r4.kicad_prl 	modified:   dipext-pin_r4/dipext-pin_r4.kicad_pro 	modified:   dipext-pin_r5/dipext-pin_r4.kicad_prl 	modified:   dipext-pin_r5/dipext-pin_r4.kicad_pro 	modified:   dipext-pin_r5/dipext-pin_r4.kicad_sch 	modified:   simpleprobecard/Gerbers.zip 	modified:   simpleprobecard/Gerbers/simpleprobecard-B_Cu.gbr 	modified:   simpleprobecard/Gerbers/simpleprobecard-B_Mask.gbr 	modified:   simpleprobecard/Gerbers/simpleprobecard-B_Paste.gbr 	modified:   simpleprobecard/Gerbers/simpleprobecard-B_Silkscreen.gbr 	modified:   simpleprobecard/Gerbers/simpleprobecard-Edge_Cuts.gbr 	modified:   simpleprobecard/Gerbers/simpleprobecard-F_Cu.gbr 	modified:   simpleprobecard/Gerbers/simpleprobecard-F_Mask.gbr 	modified:   simpleprobecard/Gerbers/simpleprobecard-F_Paste.gbr 	modified:   simpleprobecard/Gerbers/simpleprobecard-F_Silkscreen.gbr 	modified:   simpleprobecard/Gerbers/simpleprobecard-NPTH-drl_map.ps 	modified:   simpleprobecard/Gerbers/simpleprobecard-NPTH.drl 	modified:   simpleprobecard/Gerbers/simpleprobecard-PTH-drl_map.ps 	modified:   simpleprobecard/Gerbers/simpleprobecard-PTH.drl 	modified:   simpleprobecard/Gerbers/simpleprobecard-job.gbrjob 	modified:   simpleprobecard/fp-info-cache 	modified:   simpleprobecard/simpleprobecard.kicad_pcb 	modified:   simpleprobecard/simpleprobecard.kicad_pro 	modified:   simpleprobecard/simpleprobecard.kicad_sch
Parts:
- added J3: Conn_02x20_Odd_Even, Connector_IDC:IDC-Header_2x20_P2.54mm_Latch_Vertical, symbol Connector_Generic:Conn_02x20_Odd_Even
Connections:
- net P1: now reaches J1.1 (Pin_1), J2.1 (Pin_1)
- net P1: now also J3.1 (Pin_1)
- net P10: now reaches J1.10 (Pin_10), J2.10 (Pin_10)
- net P10: now also J3.19 (Pin_19)
- net P11: now reaches J1.11 (Pin_11), J2.11 (Pin_11)
- net P11: now also J3.21 (Pin_21)
- net P12: now reaches J1.12 (Pin_12), J2.12 (Pin_12)
- net P12: now also J3.23 (Pin_23)
- net P13: now reaches J1.13 (Pin_13), J2.13 (Pin_13)
- net P13: now also J3.25 (Pin_25)
- net P14: now reaches J1.14 (Pin_14), J2.14 (Pin_14)
- net P14: now also J3.27 (Pin_27)
- net P15: now reaches J1.15 (Pin_15), J2.15 (Pin_15)
- net P15: now also J3.29 (Pin_29)
- net P16: now reaches J1.16 (Pin_16), J2.16 (Pin_16)
- net P16: now also J3.31 (Pin_31)
- net P17: now reaches J1.17 (Pin_17), J2.17 (Pin_17)
- net P17: now also J3.33 (Pin_33)
- net P18: now reaches J1.18 (Pin_18), J2.18 (Pin_18)
- net P18: now also J3.35 (Pin_35)
- net P19: now reaches J1.19 (Pin_19), J2.19 (Pin_19)
- net P19: now also J3.37 (Pin_37)
- net P2: now reaches J1.2 (Pin_2), J2.2 (Pin_2)
- net P2: now also J3.3 (Pin_3)
- net P20: now reaches J1.20 (Pin_20), J2.20 (Pin_20)
- net P20: now also J3.39 (Pin_39)
- net P21: now reaches J1.21 (Pin_21), J2.21 (Pin_21)
- net P21: now also J3.40 (Pin_40)
- net P22: now reaches J1.22 (Pin_22), J2.22 (Pin_22)
- net P22: now also J3.38 (Pin_38)
- net P23: now reaches J1.23 (Pin_23), J2.23 (Pin_23)
- net P23: now also J3.36 (Pin_36)
- net P24: now reaches J1.24 (Pin_24), J2.24 (Pin_24)
- net P24: now also J3.34 (Pin_34)
- net P25: now reaches J1.25 (Pin_25), J2.25 (Pin_25)
- net P25: now also J3.32 (Pin_32)
- net P26: now reaches J1.26 (Pin_26), J2.26 (Pin_26)
- net P26: now also J3.30 (Pin_30)
- net P27: now reaches J1.27 (Pin_27), J2.27 (Pin_27)
- net P27: now also J3.28 (Pin_28)
- net P28: now reaches J1.28 (Pin_28), J2.28 (Pin_28)
- net P28: now also J3.26 (Pin_26)
- net P29: now reaches J1.29 (Pin_29), J2.29 (Pin_29)
- net P29: now also J3.24 (Pin_24)
- net P3: now reaches J1.3 (Pin_3), J2.3 (Pin_3)
- net P3: now also J3.5 (Pin_5)
- net P30: now reaches J1.30 (Pin_30), J2.30 (Pin_30)
- net P30: now also J3.22 (Pin_22)
- net P31: now reaches J1.31 (Pin_31), J2.31 (Pin_31)
- net P31: now also J3.20 (Pin_20)
- net P32: now reaches J1.32 (Pin_32), J2.32 (Pin_32)
- net P32: now also J3.18 (Pin_18)
- net P33: now reaches J1.33 (Pin_33), J2.33 (Pin_33)
- net P33: now also J3.16 (Pin_16)
- net P34: now reaches J1.34 (Pin_34), J2.34 (Pin_34)
- net P34: now also J3.14 (Pin_14)
- net P35: now reaches J1.35 (Pin_35), J2.35 (Pin_35)
- net P35: now also J3.12 (Pin_12)
- net P36: now reaches J1.36 (Pin_36), J2.36 (Pin_36)
- net P36: now also J3.10 (Pin_10)
- net P37: now reaches J1.37 (Pin_37), J2.37 (Pin_37)
- net P37: now also J3.8 (Pin_8)
- net P38: now reaches J1.38 (Pin_38), J2.38 (Pin_38)
- net P38: now also J3.6 (Pin_6)
- net P39: now reaches J1.39 (Pin_39), J2.39 (Pin_39)
- net P39: now also J3.4 (Pin_4)
- net P4: now reaches J1.4 (Pin_4), J2.4 (Pin_4)
- net P4: now also J3.7 (Pin_7)
- net P40: now reaches J1.40 (Pin_40), J2.40 (Pin_40)
- net P40: now also J3.2 (Pin_2)
- net P5: now reaches J1.5 (Pin_5), J2.5 (Pin_5)
- net P5: now also J3.9 (Pin_9)
- net P6: now reaches J1.6 (Pin_6), J2.6 (Pin_6)
- net P6: now also J3.11 (Pin_11)
- net P7: now reaches J1.7 (Pin_7), J2.7 (Pin_7)
- net P7: now also J3.13 (Pin_13)
- net P8: now reaches J1.8 (Pin_8), J2.8 (Pin_8)
- net P8: now also J3.15 (Pin_15)
- net P9: now reaches J1.9 (Pin_9), J2.9 (Pin_9)
- net P9: now also J3.17 (Pin_17)
Other:
- moved on the sheet: J2
