File: dipext-pin_r6/dipext-pin_r4.kicad_pcb (KiCad board)
At the start: 2 copper layers, 88.9 x 88.9 mm, 20 parts, among them J1 ZIF, J2 IDC40, J3 Conn_02x20_Odd_Even, J4 Conn_02x20_Odd_Even, J5 01x20, J6 01x20, J7 01x20, J8 01x20

Commit message: dipext-pin_r6: simplify mounting holes
Signed-off-by: John McMaster <johndmcmaster@gmail.com>
Parts:
- removed MK10, MK11, MK2, MK3, MK5, MK6, MK7, MK8: Mounting_Hole, Mounting_Holes:MountingHole_8.4mm_M8
Other:
- board text added: "DIP40EXT-PIN R6 © 2021 Labsmore LLC"
- board text removed: "DIP40EXT-PIN R6"
- board text removed: "© 2021 Labsmore LLC"
