File: dipext-sock_r3/dipext-pin.kicad_sch (KiCad schematic)
At the start: 8 parts, among them J1 ZIF, J2 IDC40, J3 Conn_02x20_Odd_Even, J4 Conn_02x20_Odd_Even, J5 01x20, J6 01x20, J7 01x20, J8 01x20

Commit message: Fixing schematic info block.
Other:
- title: Dipext_pin -> Dipext_sock
Changed lines of the file:
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@@
   (paper "A3")
   (title_block
-    (title "Dipext_pin")
+    (title "Dipext_sock")
     (date "2021-08-28")
-    (rev "R6")
+    (rev "R3")
   )
   (junction (at 124.46 45.72) (diameter 1.016) (color 0 0 0 0))
